File: BLEZap.sch (KiCad schematic (older format))
At the start: 10 parts, among them J1 NRJ4HF, P1 PRG_HEADER, P2 INPUT_HEADER, Q1 IRLML6344, U1 Core51822B

Commit message: SP4020 Fix
Changed lines of the file:
@@
 LIBS:modules
 LIBS:KevinsLib
-LIBS:w_connectors
 LIBS:BLEZap-cache
 EELAYER 25 0
@@
 	1    0    0    -1
 $EndComp
-$Comp
-L SP4020 D1
-U 1 1 5864C2CF
-P 4150 5050
-F 0 "D1" H 4650 4950 60  0000 C CNN
-F 1 "SP4020" H 4700 5050 60  0000 C CNN
-F 2 "" H 4100 4850 60  0001 C CNN
-F 3 "" H 4100 4850 60  0001 C CNN
-	1    4150 5050
-	1    0    0    -1
-$EndComp
 Wire Wire Line
 	5000 2800 5100 2800
@@
 L GND #PWR01
 U 1 1 58656B12
-P 4150 5700
-F 0 "#PWR01" H 4150 5450 50  0001 C CNN
-F 1 "GND" H 4150 5550 50  0000 C CNN
-F 2 "" H 4150 5700 50  0000 C CNN
-F 3 "" H 4150 5700 50  0000 C CNN
-	1    4150 5700
-	1    0    0    -1
-$EndComp
-Wire Wire Line
-	4150 5700 4150 5600
-Wire Wire Line
-	4150 4550 4150 4100
+P 4150 5250
+F 0 "#PWR01" H 4150 5000 50  0001 C CNN
+F 1 "GND" H 4150 5100 50  0000 C CNN
+F 2 "" H 4150 5250 50  0000 C CNN
+F 3 "" H 4150 5250 50  0000 C CNN
+	1    4150 5250
+	1    0    0    -1
+$EndComp
 $Comp
 L GND #PWR02
@@
 	5300 5250 5300 5350
 Wire Wire Line
-	5350 5100 4950 5100
+	4950 5100 5350 5100
 Wire Wire Line
 	4950 5100 4950 4400
-Wire Wire Line
-	4950 4400 4150 4400
-Connection ~ 4150 4400
 NoConn ~ 3750 2500
 NoConn ~ 3850 2500
@@
 Connection ~ 1450 3750
 Wire Wire Line
-	3400 3200 2900 3200
+	2900 3200 3400 3200
 Wire Wire Line
 	2900 3200 2900 3250
@@
 U 1 1 5865AEBC
 P 5150 4750
-F 0 "R2" V 5150 4750 50  0000 C CNN
+F 0 "R2" V 5250 4750 50  0000 C CNN
 F 1 "10R3" V 5150 4750 50  0000 C CNN
 F 2 "" V 5080 4750 50  0000 C CNN
@@
 Wire Wire Line
 	5600 3000 5600 2950
+$Comp
+L SP4020 D1
+U 1 1 5866A0AA
+P 4150 4850
+F 0 "D1" H 4270 4760 60  0000 C CNN
+F 1 "SP4020" H 4390 4930 60  0000 C CNN
+F 2 "" H 4100 4650 60  0001 C CNN
+F 3 "" H 4100 4650 60  0001 C CNN
+	1    4150 4850
+	1    0    0    -1
+$EndComp
+Wire Wire Line
+	4150 4100 4150 4500
+Wire Wire Line
+	4150 5250 4150 5200
+Wire Wire Line
+	4950 4400 4150 4400
+Connection ~ 4150 4400
 $EndSCHEMATC

Commit message: PCB Attempt
Parts:
- removed J1: NRJ4HF, symbol NRJ4HF
- added JP1, JP2: Jumper, Resistors_SMD:R_1206, symbol Jumper
- added P3: CONN_01X02, Pin_Headers:Pin_Header_Angled_1x02, symbol CONN_01X02
- D1: footprint (none) -> Diodes_SMD:SOD-323
- P1: footprint (none) -> KevinLibrary:POGO_PIN_PAD_1X4
- P2: footprint (none) -> KevinLibrary:Pin_Header_Straight_1x04_HB
- R1, R2, R3, R4: footprint (none) -> Resistors_SMD:R_0805
- U1: footprint (none) -> KevinLibrary:CORE51822B
Connections:
- wire segments 48 -> 51
- no-connect marks 25 -> 23
Changed lines of the file:
@@
 LIBS:valves
 LIBS:nordicsemi
-LIBS:modules
 LIBS:KevinsLib
 LIBS:BLEZap-cache
@@
 F 0 "P2" H 7000 4550 50  0000 C CNN
 F 1 "INPUT_HEADER" V 7100 4300 50  0000 C CNN
-F 2 "" H 7000 4300 50  0000 C CNN
+F 2 "KevinLibrary:Pin_Header_Straight_1x04_HB" H 7000 4300 50  0001 C CNN
 F 3 "" H 7000 4300 50  0000 C CNN
 	1    7000 4300
@@
 F 0 "P1" H 7000 3500 50  0000 C CNN
 F 1 "PRG_HEADER" V 7100 3250 50  0000 C CNN
-F 2 "" H 7000 3250 50  0000 C CNN
+F 2 "KevinLibrary:POGO_PIN_PAD_1X4" H 7000 3250 50  0001 C CNN
 F 3 "" H 7000 3250 50  0000 C CNN
 	1    7000 3250
@@
 F 0 "U1" H 3450 2800 60  0000 C CNN
 F 1 "Core51822B" H 4200 3300 60  0000 C CNN
-F 2 "" H 3800 2850 60  0001 C CNN
+F 2 "KevinLibrary:CORE51822B" H 3800 2850 60  0001 C CNN
 F 3 "" H 3800 2850 60  0001 C CNN
 	1    4200 3300
@@
 F 0 "R1" V 1530 3950 50  0000 C CNN
 F 1 "100R" V 1450 3950 50  0000 C CNN
-F 2 "" V 1380 3950 50  0000 C CNN
+F 2 "Resistors_SMD:R_0805" V 1380 3950 50  0001 C CNN
 F 3 "" H 1450 3950 50  0000 C CNN
 	1    1450 3950
@@
 L GNDD #PWR06
 U 1 1 58656F52
-P 1850 4500
-F 0 "#PWR06" H 1850 4250 50  0001 C CNN
-F 1 "GNDD" H 1850 4350 50  0000 C CNN
-F 2 "" H 1850 4500 50  0000 C CNN
-F 3 "" H 1850 4500 50  0000 C CNN
-	1    1850 4500
+P 2350 4500
+F 0 "#PWR06" H 2350 4250 50  0001 C CNN
+F 1 "GNDD" H 2350 4350 50  0000 C CNN
+F 2 "" H 2350 4500 50  0000 C CNN
+F 3 "" H 2350 4500 50  0000 C CNN
+	1    2350 4500
 	1    0    0    -1
 $EndComp
@@
 	1150 4350 1150 4500
 Wire Wire Line
-	1700 4450 1850 4450
-Wire Wire Line
-	1850 4350 1850 4500
+	2350 4350 2350 4500
 $Comp
 L GNDD #PWR07
@@
 	3200 3000 3200 2900
 $Comp
-L NRJ4HF J1
-U 1 1 586574DE
-P 6050 5100
-F 0 "J1" H 6050 4850 60  0000 C CNN
-F 1 "NRJ4HF" H 6100 5350 60  0000 C CNN
-F 2 "" H 6050 5100 60  0001 C CNN
-F 3 "" H 6050 5100 60  0001 C CNN
-	1    6050 5100
-	-1   0    0    1
-$EndComp
-NoConn ~ 5350 5050
-NoConn ~ 5350 5200
-$Comp
 L GNDD #PWR010
 U 1 1 58657574
@@
 $EndComp
 Wire Wire Line
-	5350 5250 5300 5250
-Wire Wire Line
-	5300 5250 5300 5350
-Wire Wire Line
-	4950 5100 5350 5100
+	5300 5200 5300 5350
+Wire Wire Line
+	4950 5100 5500 5100
 Wire Wire Line
 	4950 5100 4950 4400
@@
 L PWR_FLAG #FLG011
 U 1 1 58657A0B
-P 1850 4350
-F 0 "#FLG011" H 1850 4445 50  0001 C CNN
-F 1 "PWR_FLAG" H 1850 4530 50  0000 C CNN
-F 2 "" H 1850 4350 50  0000 C CNN
-F 3 "" H 1850 4350 50  0000 C CNN
-	1    1850 4350
-	1    0    0    -1
-$EndComp
-Connection ~ 1850 4450
+P 2350 4350
+F 0 "#FLG011" H 2350 4445 50  0001 C CNN
+F 1 "PWR_FLAG" H 2350 4530 50  0000 C CNN
+F 2 "" H 2350 4350 50  0000 C CNN
+F 3 "" H 2350 4350 50  0000 C CNN
+	1    2350 4350
+	1    0    0    -1
+$EndComp
+Connection ~ 2350 4450
 Connection ~ 1150 4450
 Wire Wire Line
@@
 F 0 "R4" V 5430 2400 50  0000 C CNN
 F 1 "10R3" V 5350 2400 50  0000 C CNN
-F 2 "" V 5280 2400 50  0000 C CNN
+F 2 "Resistors_SMD:R_0805" V 5280 2400 50  0001 C CNN
 F 3 "" H 5350 2400 50  0000 C CNN
 	1    5350 2400
@@
 F 0 "R3" V 5380 3000 50  0000 C CNN
 F 1 "10R3" V 5300 3000 50  0000 C CNN
-F 2 "" V 5230 3000 50  0000 C CNN
+F 2 "Resistors_SMD:R_0805" V 5230 3000 50  0001 C CNN
 F 3 "" H 5300 3000 50  0000 C CNN
 	1    5300 3000
@@
 F 0 "R2" V 5250 4750 50  0000 C CNN
 F 1 "10R3" V 5150 4750 50  0000 C CNN
-F 2 "" V 5080 4750 50  0000 C CNN
+F 2 "Resistors_SMD:R_0805" V 5080 4750 50  0001 C CNN
 F 3 "" H 5150 4750 50  0000 C CNN
 	1    5150 4750
@@
 F 0 "D1" H 4270 4760 60  0000 C CNN
 F 1 "SP4020" H 4390 4930 60  0000 C CNN
-F 2 "" H 4100 4650 60  0001 C CNN
+F 2 "Diodes_SMD:SOD-323" H 4100 4650 60  0001 C CNN
 F 3 "" H 4100 4650 60  0001 C CNN
 	1    4150 4850
@@
 Wire Wire Line
 	4150 5250 4150 5200
-Wire Wire Line
-	4950 4400 4150 4400
 Connection ~ 4150 4400
+$Comp
+L CONN_01X02 P3
+U 1 1 58697198
+P 5700 5150
+F 0 "P3" H 5700 5300 50  0000 C CNN
+F 1 "CONN_01X02" V 5800 5150 50  0000 C CNN
+F 2 "Pin_Headers:Pin_Header_Angled_1x02" H 5700 5150 50  0001 C CNN
+F 3 "" H 5700 5150 50  0000 C CNN
+	1    5700 5150
+	1    0    0    -1
+$EndComp
+Wire Wire Line
+	5500 5200 5300 5200
+$Comp
+L Jumper JP1
+U 1 1 586993E3
+P 2050 4450
+F 0 "JP1" H 2050 4600 50  0000 C CNN
+F 1 "Jumper" H 2050 4370 50  0000 C CNN
+F 2 "Resistors_SMD:R_1206" H 2050 4450 50  0001 C CNN
+F 3 "" H 2050 4450 50  0000 C CNN
+	1    2050 4450
+	1    0    0    -1
+$EndComp
+Wire Wire Line
+	1700 4450 1750 4450
+$Comp
+L Jumper JP2
+U 1 1 586996CD
+P 4550 4400
+F 0 "JP2" H 4550 4550 50  0000 C CNN
+F 1 "Jumper" H 4550 4320 50  0000 C CNN
+F 2 "Resistors_SMD:R_1206" H 4550 4400 50  0001 C CNN
+F 3 "" H 4550 4400 50  0000 C CNN
+	1    4550 4400
+	1    0    0    -1
+$EndComp
+Wire Wire Line
+	4950 4400 4850 4400
+Wire Wire Line
+	4150 4400 4250 4400
+$Comp
+L GNDD #PWR018
+U 1 1 58699CDB
+P 1800 4550
+F 0 "#PWR018" H 1800 4300 50  0001 C CNN
+F 1 "GNDD" H 1800 4400 50  0000 C CNN
+F 2 "" H 1800 4550 50  0000 C CNN
+F 3 "" H 1800 4550 50  0000 C CNN
+	1    1800 4550
+	1    0    0    -1
+$EndComp
+Wire Wire Line
+	1800 4550 1750 4550
+Wire Wire Line
+	1750 4550 1750 4450
 $EndSCHEMATC

Commit message: PCB Ready
Parts:
- removed JP1, JP2: Jumper, Resistors_SMD:R_1206, symbol Jumper
- P1: footprint KevinLibrary:POGO_PIN_PAD_1X4 -> Pin_Headers:Pin_Header_Straight_1x04
- P2: footprint KevinLibrary:Pin_Header_Straight_1x04_HB -> Pin_Headers:Pin_Header_Straight_1x04
Connections:
- wire segments 51 -> 48
Changed lines of the file:
@@
 F 0 "P2" H 7000 4550 50  0000 C CNN
 F 1 "INPUT_HEADER" V 7100 4300 50  0000 C CNN
-F 2 "KevinLibrary:Pin_Header_Straight_1x04_HB" H 7000 4300 50  0001 C CNN
+F 2 "Pin_Headers:Pin_Header_Straight_1x04" H 7000 4300 50  0001 C CNN
 F 3 "" H 7000 4300 50  0000 C CNN
 	1    7000 4300
@@
 F 0 "P1" H 7000 3500 50  0000 C CNN
 F 1 "PRG_HEADER" V 7100 3250 50  0000 C CNN
-F 2 "KevinLibrary:POGO_PIN_PAD_1X4" H 7000 3250 50  0001 C CNN
+F 2 "Pin_Headers:Pin_Header_Straight_1x04" H 7000 3250 50  0001 C CNN
 F 3 "" H 7000 3250 50  0000 C CNN
 	1    7000 3250
@@
 L GNDD #PWR06
 U 1 1 58656F52
-P 2350 4500
-F 0 "#PWR06" H 2350 4250 50  0001 C CNN
-F 1 "GNDD" H 2350 4350 50  0000 C CNN
-F 2 "" H 2350 4500 50  0000 C CNN
-F 3 "" H 2350 4500 50  0000 C CNN
-	1    2350 4500
+P 2000 4500
+F 0 "#PWR06" H 2000 4250 50  0001 C CNN
+F 1 "GNDD" H 2000 4350 50  0000 C CNN
+F 2 "" H 2000 4500 50  0000 C CNN
+F 3 "" H 2000 4500 50  0000 C CNN
+	1    2000 4500
 	1    0    0    -1
 $EndComp
@@
 Wire Wire Line
 	1150 4350 1150 4500
-Wire Wire Line
-	2350 4350 2350 4500
 $Comp
 L GNDD #PWR07
@@
 	4950 5100 5500 5100
 Wire Wire Line
-	4950 5100 4950 4400
+	4950 4400 4950 5100
 NoConn ~ 3750 2500
 NoConn ~ 3850 2500
@@
 L PWR_FLAG #FLG011
 U 1 1 58657A0B
-P 2350 4350
-F 0 "#FLG011" H 2350 4445 50  0001 C CNN
-F 1 "PWR_FLAG" H 2350 4530 50  0000 C CNN
-F 2 "" H 2350 4350 50  0000 C CNN
-F 3 "" H 2350 4350 50  0000 C CNN
-	1    2350 4350
-	1    0    0    -1
-$EndComp
-Connection ~ 2350 4450
+P 2000 4350
+F 0 "#FLG011" H 2000 4445 50  0001 C CNN
+F 1 "PWR_FLAG" H 2000 4530 50  0000 C CNN
+F 2 "" H 2000 4350 50  0000 C CNN
+F 3 "" H 2000 4350 50  0000 C CNN
+	1    2000 4350
+	1    0    0    -1
+$EndComp
 Connection ~ 1150 4450
 Wire Wire Line
@@
 Wire Wire Line
 	5500 5200 5300 5200
-$Comp
-L Jumper JP1
-U 1 1 586993E3
-P 2050 4450
-F 0 "JP1" H 2050 4600 50  0000 C CNN
-F 1 "Jumper" H 2050 4370 50  0000 C CNN
-F 2 "Resistors_SMD:R_1206" H 2050 4450 50  0001 C CNN
-F 3 "" H 2050 4450 50  0000 C CNN
-	1    2050 4450
-	1    0    0    -1
-$EndComp
-Wire Wire Line
-	1700 4450 1750 4450
-$Comp
-L Jumper JP2
-U 1 1 586996CD
-P 4550 4400
-F 0 "JP2" H 4550 4550 50  0000 C CNN
-F 1 "Jumper" H 4550 4320 50  0000 C CNN
-F 2 "Resistors_SMD:R_1206" H 4550 4400 50  0001 C CNN
-F 3 "" H 4550 4400 50  0000 C CNN
-	1    4550 4400
-	1    0    0    -1
-$EndComp
-Wire Wire Line
-	4950 4400 4850 4400
-Wire Wire Line
-	4150 4400 4250 4400
-$Comp
-L GNDD #PWR018
-U 1 1 58699CDB
-P 1800 4550
-F 0 "#PWR018" H 1800 4300 50  0001 C CNN
-F 1 "GNDD" H 1800 4400 50  0000 C CNN
-F 2 "" H 1800 4550 50  0000 C CNN
-F 3 "" H 1800 4550 50  0000 C CNN
-	1    1800 4550
-	1    0    0    -1
-$EndComp
-Wire Wire Line
-	1800 4550 1750 4550
-Wire Wire Line
-	1750 4550 1750 4450
+Wire Wire Line
+	4150 4400 4950 4400
+Wire Wire Line
+	2000 4350 2000 4500
+Wire Wire Line
+	1700 4450 2000 4450
+Connection ~ 2000 4450
 $EndSCHEMATC

Commit message: SWD Swap
Connections:
- net SWCLK: now also P1.3 (P3); no longer P1.2 (P2)
- net SWDIO: now also P1.2 (P2); no longer P1.3 (P3)
Changed lines of the file:
@@
 	6800 3300 6500 3300
 Text Label 6500 3200 0    60   ~ 0
+SWDIO
+Text Label 6500 3300 0    60   ~ 0
 SWCLK
-Text Label 6500 3300 0    60   ~ 0
-SWDIO
 $Comp
 L GND #PWR01

Commit message: Protection Diode
Parts:
- added D?: 1N5819, symbol D
Connections:
- net CFG_BTN: now also P2.1 (P1); no longer P2.3 (P3)
- net RELAY: now also P2.3 (P3), D?.1 (K); no longer P2.2 (P2), U1.24 (P10)
- net VDD: now also P2.2 (P2); no longer P2.1 (P1)
- new net: D?.2 (A), U1.24 (P10)
Changed lines of the file:
@@
 	5000 2800 5100 2800
 Wire Wire Line
-	5100 2400 5100 2900
+	5100 2400 5100 2800
+Wire Wire Line
+	5100 2800 5100 2900
 Wire Wire Line
 	5100 2900 5000 2900
@@
 $EndComp
 Wire Wire Line
-	6800 4150 6650 4150
-Wire Wire Line
-	6650 4150 6650 4050
-Wire Wire Line
 	6800 4450 6650 4450
 Wire Wire Line
 	6650 4450 6650 4500
 Wire Wire Line
-	5000 3800 5400 3800
-Text Label 5400 3800 2    60   ~ 0
+	5000 3800 5150 3800
+Text Label 5700 3800 2    60   ~ 0
 RELAY
 Wire Wire Line
-	6800 4250 6400 4250
-Text Label 6400 4250 0    60   ~ 0
+	6300 4250 6800 4250
+Text Label 6400 4350 0    60   ~ 0
 RELAY
 Wire Wire Line
@@
 Text Label 5400 3700 2    60   ~ 0
 CFG_BTN
-Text Label 6400 4350 0    60   ~ 0
+Text Label 6400 4150 0    60   ~ 0
 CFG_BTN
 $Comp
@@
 $EndComp
 Wire Wire Line
-	1450 3650 1450 3800
+	1450 3650 1450 3750
+Wire Wire Line
+	1450 3750 1450 3800
 Wire Wire Line
 	1450 4100 1450 4150
@@
 	1300 4450 1150 4450
 Wire Wire Line
-	1150 4350 1150 4500
+	1150 4350 1150 4450
+Wire Wire Line
+	1150 4450 1150 4500
 $Comp
 L GNDD #PWR07
@@
 	5300 5200 5300 5350
 Wire Wire Line
-	4950 5100 5500 5100
+	4950 5100 5150 5100
+Wire Wire Line
+	5150 5100 5500 5100
 Wire Wire Line
 	4950 4400 4950 5100
@@
 Connection ~ 1450 3750
 Wire Wire Line
-	2900 3200 3400 3200
+	2900 3200 3200 3200
+Wire Wire Line
+	3200 3200 3400 3200
 Wire Wire Line
 	2900 3200 2900 3250
@@
 L VDD #PWR012
 U 1 1 58657E30
-P 6650 4050
-F 0 "#PWR012" H 6650 3900 50  0001 C CNN
-F 1 "VDD" H 6650 4200 50  0000 C CNN
-F 2 "" H 6650 4050 50  0000 C CNN
-F 3 "" H 6650 4050 50  0000 C CNN
-	1    6650 4050
+P 6300 4200
+F 0 "#PWR012" H 6300 4050 50  0001 C CNN
+F 1 "VDD" H 6300 4350 50  0000 C CNN
+F 2 "" H 6300 4200 50  0000 C CNN
+F 3 "" H 6300 4200 50  0000 C CNN
+	1    6300 4200
 	1    0    0    -1
 $EndComp
@@
 $EndComp
 Wire Wire Line
-	4150 4100 4150 4500
+	4150 4100 4150 4400
+Wire Wire Line
+	4150 4400 4150 4500
 Wire Wire Line
 	4150 5250 4150 5200
@@
 	4150 4400 4950 4400
 Wire Wire Line
-	2000 4350 2000 4500
+	2000 4350 2000 4450
+Wire Wire Line
+	2000 4450 2000 4500
 Wire Wire Line
 	1700 4450 2000 4450
 Connection ~ 2000 4450
+Wire Wire Line
+	6800 4150 6400 4150
+Wire Wire Line
+	6300 4250 6300 4200
+$Comp
+L D D?
+U 1 1 58901F7D
+P 5300 3800
+F 0 "D?" H 5300 3900 50  0000 C CNN
+F 1 "1N5819" H 5300 4000 50  0000 C CNN
+F 2 "" H 5300 3800 50  0000 C CNN
+F 3 "" H 5300 3800 50  0000 C CNN
+	1    5300 3800
+	-1   0    0    1
+$EndComp
+Wire Wire Line
+	5450 3800 5700 3800
 $EndSCHEMATC
