File: BLEZap.sch (KiCad schematic (older format))
At the start: 11 parts, among them P1 PRG_HEADER, P2 INPUT_HEADER, P3 CONN_01X02, Q1 IRLML6344, U1 Core51822B

Commit message: Version 2
Parts:
- removed Q1: IRLML6344, TO_SOT_Packages_SMD:SOT-23, symbol IRLML6344
- removed R1: 100R, Resistors_SMD:R_0805, symbol R
- added U2: MP1584_MOD, KevinLibrary:MP1584_MOD_ALL_UNDER, symbol MP1584_MOD
- D2: renamed from D?; footprint (none) -> Diodes_SMD:D_0805
Connections:
- net GNDD is gone; now on net GND: P1.4 (P4), P3.2 (P2), R4.1, U1.1 (GND), U1.11 (GND)
- net GND: now also U2.1 (OUT-), U2.5 (IN-)
- net VDD: now also U2.4 (OUT+); no longer P2.2 (P2)
- new net +24V: P2.2 (P2), U2.8 (IN+)
Changed lines of the file:
@@
 	5000 2800 5100 2800
 Wire Wire Line
-	5100 2400 5100 2800
-Wire Wire Line
-	5100 2800 5100 2900
+	5100 2400 5100 2900
 Wire Wire Line
 	5100 2900 5000 2900
 Connection ~ 5100 2800
-$Comp
-L IRLML6344 Q1
-U 1 1 5865689C
-P 1500 4350
-F 0 "Q1" V 1400 4400 50  0000 L CNN
-F 1 "IRLML6344" V 1700 4150 50  0000 L CNN
-F 2 "TO_SOT_Packages_SMD:SOT-23" H 1600 4325 50  0001 L CIN
-F 3 "" H 1400 4400 50  0000 L CNN
-	1    1500 4350
-	0    1    1    0
-$EndComp
 Wire Wire Line
 	3400 3400 3150 3400
@@
 L PWR_FLAG #FLG03
 U 1 1 58656D18
-P 1150 3700
-F 0 "#FLG03" H 1150 3795 50  0001 C CNN
-F 1 "PWR_FLAG" H 1150 3880 50  0000 C CNN
-F 2 "" H 1150 3700 50  0000 C CNN
-F 3 "" H 1150 3700 50  0000 C CNN
-	1    1150 3700
-	1    0    0    -1
+P 1700 2950
+F 0 "#FLG03" H 1700 3045 50  0001 C CNN
+F 1 "PWR_FLAG" H 1700 3130 50  0000 C CNN
+F 2 "" H 1700 2950 50  0000 C CNN
+F 3 "" H 1700 2950 50  0000 C CNN
+	1    1700 2950
+	0    -1   -1   0
 $EndComp
 $Comp
 L PWR_FLAG #FLG04
 U 1 1 58656D39
-P 1150 4350
-F 0 "#FLG04" H 1150 4445 50  0001 C CNN
-F 1 "PWR_FLAG" H 1150 4530 50  0000 C CNN
-F 2 "" H 1150 4350 50  0000 C CNN
-F 3 "" H 1150 4350 50  0000 C CNN
-	1    1150 4350
-	1    0    0    -1
-$EndComp
-$Comp
-L R R1
-U 1 1 58656E6F
-P 1450 3950
-F 0 "R1" V 1530 3950 50  0000 C CNN
-F 1 "100R" V 1450 3950 50  0000 C CNN
-F 2 "Resistors_SMD:R_0805" V 1380 3950 50  0001 C CNN
-F 3 "" H 1450 3950 50  0000 C CNN
-	1    1450 3950
-	1    0    0    -1
-$EndComp
-Wire Wire Line
-	1450 3650 1450 3750
-Wire Wire Line
-	1450 3750 1450 3800
-Wire Wire Line
-	1450 4100 1450 4150
+P 1700 4400
+F 0 "#FLG04" H 1700 4495 50  0001 C CNN
+F 1 "PWR_FLAG" H 1700 4580 50  0000 C CNN
+F 2 "" H 1700 4400 50  0000 C CNN
+F 3 "" H 1700 4400 50  0000 C CNN
+	1    1700 4400
+	0    -1   -1   0
+$EndComp
 $Comp
 L GND #PWR05
 U 1 1 58656F33
-P 1150 4500
-F 0 "#PWR05" H 1150 4250 50  0001 C CNN
-F 1 "GND" H 1150 4350 50  0000 C CNN
-F 2 "" H 1150 4500 50  0000 C CNN
-F 3 "" H 1150 4500 50  0000 C CNN
-	1    1150 4500
-	1    0    0    -1
-$EndComp
-$Comp
-L GNDD #PWR06
-U 1 1 58656F52
-P 2000 4500
-F 0 "#PWR06" H 2000 4250 50  0001 C CNN
-F 1 "GNDD" H 2000 4350 50  0000 C CNN
-F 2 "" H 2000 4500 50  0000 C CNN
-F 3 "" H 2000 4500 50  0000 C CNN
-	1    2000 4500
-	1    0    0    -1
-$EndComp
-Wire Wire Line
-	1300 4450 1150 4450
-Wire Wire Line
-	1150 4350 1150 4450
-Wire Wire Line
-	1150 4450 1150 4500
-$Comp
-L GNDD #PWR07
-U 1 1 58656FD5
-P 5600 2500
-F 0 "#PWR07" H 5600 2250 50  0001 C CNN
-F 1 "GNDD" H 5600 2350 50  0000 C CNN
-F 2 "" H 5600 2500 50  0000 C CNN
-F 3 "" H 5600 2500 50  0000 C CNN
-	1    5600 2500
-	1    0    0    -1
-$EndComp
-$Comp
-L GNDD #PWR08
-U 1 1 58656FFF
-P 6650 3450
-F 0 "#PWR08" H 6650 3200 50  0001 C CNN
-F 1 "GNDD" H 6650 3300 50  0000 C CNN
-F 2 "" H 6650 3450 50  0000 C CNN
-F 3 "" H 6650 3450 50  0000 C CNN
-	1    6650 3450
+P 2350 4500
+F 0 "#PWR05" H 2350 4250 50  0001 C CNN
+F 1 "GND" H 2350 4350 50  0000 C CNN
+F 2 "" H 2350 4500 50  0000 C CNN
+F 3 "" H 2350 4500 50  0000 C CNN
+	1    2350 4500
 	1    0    0    -1
 $EndComp
 Wire Wire Line
 	3200 3100 3400 3100
-$Comp
-L GNDD #PWR09
-U 1 1 58657060
-P 2900 3250
-F 0 "#PWR09" H 2900 3000 50  0001 C CNN
-F 1 "GNDD" H 2900 3100 50  0000 C CNN
-F 2 "" H 2900 3250 50  0000 C CNN
-F 3 "" H 2900 3250 50  0000 C CNN
-	1    2900 3250
-	1    0    0    -1
-$EndComp
 Wire Wire Line
 	3400 3000 3200 3000
 Wire Wire Line
 	3200 3000 3200 2900
-$Comp
-L GNDD #PWR010
-U 1 1 58657574
-P 5300 5350
-F 0 "#PWR010" H 5300 5100 50  0001 C CNN
-F 1 "GNDD" H 5300 5200 50  0000 C CNN
-F 2 "" H 5300 5350 50  0000 C CNN
-F 3 "" H 5300 5350 50  0000 C CNN
-	1    5300 5350
-	1    0    0    -1
-$EndComp
 Wire Wire Line
 	5300 5200 5300 5350
 Wire Wire Line
-	4950 5100 5150 5100
-Wire Wire Line
-	5150 5100 5500 5100
+	4950 5100 5500 5100
 Wire Wire Line
 	4950 4400 4950 5100
@@
 NoConn ~ 3750 4100
 $Comp
-L PWR_FLAG #FLG011
+L PWR_FLAG #FLG06
 U 1 1 58657A0B
-P 2000 4350
-F 0 "#FLG011" H 2000 4445 50  0001 C CNN
-F 1 "PWR_FLAG" H 2000 4530 50  0000 C CNN
-F 2 "" H 2000 4350 50  0000 C CNN
-F 3 "" H 2000 4350 50  0000 C CNN
-	1    2000 4350
-	1    0    0    -1
-$EndComp
-Connection ~ 1150 4450
-Wire Wire Line
-	1150 3750 1150 3700
-Wire Wire Line
-	1150 3750 1450 3750
-Connection ~ 1450 3750
-Wire Wire Line
-	2900 3200 3200 3200
-Wire Wire Line
-	3200 3200 3400 3200
+P 2450 4400
+F 0 "#FLG06" H 2450 4495 50  0001 C CNN
+F 1 "PWR_FLAG" H 2450 4580 50  0000 C CNN
+F 2 "" H 2450 4400 50  0000 C CNN
+F 3 "" H 2450 4400 50  0000 C CNN
+	1    2450 4400
+	0    1    1    0
+$EndComp
+Wire Wire Line
+	2900 3200 3400 3200
 Wire Wire Line
 	2900 3200 2900 3250
@@
 Connection ~ 3200 3200
 $Comp
-L VDD #PWR012
-U 1 1 58657E30
-P 6300 4200
-F 0 "#PWR012" H 6300 4050 50  0001 C CNN
-F 1 "VDD" H 6300 4350 50  0000 C CNN
-F 2 "" H 6300 4200 50  0000 C CNN
-F 3 "" H 6300 4200 50  0000 C CNN
-	1    6300 4200
-	1    0    0    -1
-$EndComp
-$Comp
-L VDD #PWR013
+L VDD #PWR07
 U 1 1 58657E66
-P 1450 3650
-F 0 "#PWR013" H 1450 3500 50  0001 C CNN
-F 1 "VDD" H 1450 3800 50  0000 C CNN
-F 2 "" H 1450 3650 50  0000 C CNN
-F 3 "" H 1450 3650 50  0000 C CNN
-	1    1450 3650
-	1    0    0    -1
-$EndComp
-$Comp
-L VDD #PWR014
+P 1800 2850
+F 0 "#PWR07" H 1800 2700 50  0001 C CNN
+F 1 "VDD" H 1800 3000 50  0000 C CNN
+F 2 "" H 1800 2850 50  0000 C CNN
+F 3 "" H 1800 2850 50  0000 C CNN
+	1    1800 2850
+	1    0    0    -1
+$EndComp
+$Comp
+L VDD #PWR08
 U 1 1 58657E95
 P 3200 2900
-F 0 "#PWR014" H 3200 2750 50  0001 C CNN
+F 0 "#PWR08" H 3200 2750 50  0001 C CNN
 F 1 "VDD" H 3200 3050 50  0000 C CNN
 F 2 "" H 3200 2900 50  0000 C CNN
@@
 $EndComp
 $Comp
-L VDD #PWR015
+L VDD #PWR09
 U 1 1 58657EE2
 P 5600 2950
-F 0 "#PWR015" H 5600 2800 50  0001 C CNN
+F 0 "#PWR09" H 5600 2800 50  0001 C CNN
 F 1 "VDD" H 5600 3100 50  0000 C CNN
 F 2 "" H 5600 2950 50  0000 C CNN
@@
 $EndComp
 $Comp
-L VDD #PWR016
+L VDD #PWR010
 U 1 1 58657F3C
 P 6650 3000
-F 0 "#PWR016" H 6650 2850 50  0001 C CNN
+F 0 "#PWR010" H 6650 2850 50  0001 C CNN
 F 1 "VDD" H 6650 3150 50  0000 C CNN
 F 2 "" H 6650 3000 50  0000 C CNN
@@
 $EndComp
 $Comp
-L VDD #PWR017
+L VDD #PWR011
 U 1 1 5865AF88
 P 5150 4450
-F 0 "#PWR017" H 5150 4300 50  0001 C CNN
+F 0 "#PWR011" H 5150 4300 50  0001 C CNN
 F 1 "VDD" H 5150 4600 50  0000 C CNN
 F 2 "" H 5150 4450 50  0000 C CNN
@@
 $EndComp
 Wire Wire Line
-	4150 4100 4150 4400
-Wire Wire Line
-	4150 4400 4150 4500
+	4150 4100 4150 4500
 Wire Wire Line
 	4150 5250 4150 5200
@@
 	4150 4400 4950 4400
 Wire Wire Line
-	2000 4350 2000 4450
-Wire Wire Line
-	2000 4450 2000 4500
-Wire Wire Line
-	1700 4450 2000 4450
-Connection ~ 2000 4450
-Wire Wire Line
 	6800 4150 6400 4150
 Wire Wire Line
 	6300 4250 6300 4200
 $Comp
-L D D?
+L D D2
 U 1 1 58901F7D
 P 5300 3800
-F 0 "D?" H 5300 3900 50  0000 C CNN
+F 0 "D2" H 5300 3900 50  0000 C CNN
 F 1 "1N5819" H 5300 4000 50  0000 C CNN
-F 2 "" H 5300 3800 50  0000 C CNN
+F 2 "Diodes_SMD:D_0805" H 5300 3800 50  0001 C CNN
 F 3 "" H 5300 3800 50  0000 C CNN
 	1    5300 3800
@@
 Wire Wire Line
 	5450 3800 5700 3800
+$Comp
+L GND #PWR012
+U 1 1 5891599C
+P 2900 3250
+F 0 "#PWR012" H 2900 3000 50  0001 C CNN
+F 1 "GND" H 2900 3100 50  0000 C CNN
+F 2 "" H 2900 3250 50  0000 C CNN
+F 3 "" H 2900 3250 50  0000 C CNN
+	1    2900 3250
+	1    0    0    -1
+$EndComp
+$Comp
+L GND #PWR013
+U 1 1 589159D5
+P 5600 2500
+F 0 "#PWR013" H 5600 2250 50  0001 C CNN
+F 1 "GND" H 5600 2350 50  0000 C CNN
+F 2 "" H 5600 2500 50  0000 C CNN
+F 3 "" H 5600 2500 50  0000 C CNN
+	1    5600 2500
+	1    0    0    -1
+$EndComp
+$Comp
+L GND #PWR014
+U 1 1 58915A68
+P 5300 5350
+F 0 "#PWR014" H 5300 5100 50  0001 C CNN
+F 1 "GND" H 5300 5200 50  0000 C CNN
+F 2 "" H 5300 5350 50  0000 C CNN
+F 3 "" H 5300 5350 50  0000 C CNN
+	1    5300 5350
+	1    0    0    -1
+$EndComp
+$Comp
+L GND #PWR015
+U 1 1 58915B1F
+P 6650 3450
+F 0 "#PWR015" H 6650 3200 50  0001 C CNN
+F 1 "GND" H 6650 3300 50  0000 C CNN
+F 2 "" H 6650 3450 50  0000 C CNN
+F 3 "" H 6650 3450 50  0000 C CNN
+	1    6650 3450
+	1    0    0    -1
+$EndComp
+$Comp
+L +24V #PWR016
+U 1 1 58915B47
+P 6300 4200
+F 0 "#PWR016" H 6300 4050 50  0001 C CNN
+F 1 "+24V" H 6300 4340 50  0000 C CNN
+F 2 "" H 6300 4200 50  0000 C CNN
+F 3 "" H 6300 4200 50  0000 C CNN
+	1    6300 4200
+	1    0    0    -1
+$EndComp
+$Comp
+L MP1584_MOD U2
+U 1 1 58915C24
+P 2100 3700
+F 0 "U2" H 2100 3550 60  0000 C CNN
+F 1 "MP1584_MOD" H 2100 3850 60  0000 C CNN
+F 2 "KevinLibrary:MP1584_MOD_ALL_UNDER" H 2100 3700 60  0001 C CNN
+F 3 "" H 2100 3700 60  0001 C CNN
+	1    2100 3700
+	1    0    0    -1
+$EndComp
+$Comp
+L +24V #PWR017
+U 1 1 58915CC9
+P 1800 4500
+F 0 "#PWR017" H 1800 4350 50  0001 C CNN
+F 1 "+24V" H 1800 4640 50  0000 C CNN
+F 2 "" H 1800 4500 50  0000 C CNN
+F 3 "" H 1800 4500 50  0000 C CNN
+	1    1800 4500
+	-1   0    0    1
+$EndComp
+$Comp
+L GND #PWR018
+U 1 1 58915DF8
+P 2550 3000
+F 0 "#PWR018" H 2550 2750 50  0001 C CNN
+F 1 "GND" H 2550 2850 50  0000 C CNN
+F 2 "" H 2550 3000 50  0000 C CNN
+F 3 "" H 2550 3000 50  0000 C CNN
+	1    2550 3000
+	1    0    0    -1
+$EndComp
+Wire Wire Line
+	2350 3000 2350 2900
+Wire Wire Line
+	2350 2900 2550 2900
+Wire Wire Line
+	2550 2900 2550 3000
+Wire Wire Line
+	1800 2850 1800 3000
+Wire Wire Line
+	1800 4300 1800 4500
+Wire Wire Line
+	2350 4300 2350 4500
+Wire Wire Line
+	1700 2950 1800 2950
+Connection ~ 1800 2950
+Wire Wire Line
+	1700 4400 1800 4400
+Connection ~ 1800 4400
+Wire Wire Line
+	2450 4400 2350 4400
+Connection ~ 2350 4400
 $EndSCHEMATC

Commit message: LP Filter
Parts:
- added C1: .1uF, Capacitors_SMD:C_0805, symbol C
- added R1: 10R4, Resistors_SMD:R_0805, symbol R
- R2, R3, R4: value 10R3 -> 10R4
Connections:
- net GND: now also C1.2
- net at D1.1, R2.2, U1.29 (P15): now also C1.1, R1.2; no longer P3.1 (P1)
- new net: P3.1 (P1), R1.1
Other:
- moved on the sheet: P3
Changed lines of the file:
@@
 	3200 3000 3200 2900
 Wire Wire Line
-	5300 5200 5300 5350
-Wire Wire Line
-	4950 5100 5500 5100
+	5400 5400 6250 5400
+Wire Wire Line
+	4950 5100 5850 5100
 Wire Wire Line
 	4950 4400 4950 5100
@@
 P 5350 2400
 F 0 "R4" V 5430 2400 50  0000 C CNN
-F 1 "10R3" V 5350 2400 50  0000 C CNN
+F 1 "10R4" V 5350 2400 50  0000 C CNN
 F 2 "Resistors_SMD:R_0805" V 5280 2400 50  0001 C CNN
 F 3 "" H 5350 2400 50  0000 C CNN
@@
 P 5300 3000
 F 0 "R3" V 5380 3000 50  0000 C CNN
-F 1 "10R3" V 5300 3000 50  0000 C CNN
+F 1 "10R4" V 5300 3000 50  0000 C CNN
 F 2 "Resistors_SMD:R_0805" V 5230 3000 50  0001 C CNN
 F 3 "" H 5300 3000 50  0000 C CNN
@@
 P 5150 4750
 F 0 "R2" V 5250 4750 50  0000 C CNN
-F 1 "10R3" V 5150 4750 50  0000 C CNN
+F 1 "10R4" V 5150 4750 50  0000 C CNN
 F 2 "Resistors_SMD:R_0805" V 5080 4750 50  0001 C CNN
 F 3 "" H 5150 4750 50  0000 C CNN
@@
 L CONN_01X02 P3
 U 1 1 58697198
-P 5700 5150
-F 0 "P3" H 5700 5300 50  0000 C CNN
-F 1 "CONN_01X02" V 5800 5150 50  0000 C CNN
-F 2 "Pin_Headers:Pin_Header_Angled_1x02" H 5700 5150 50  0001 C CNN
-F 3 "" H 5700 5150 50  0000 C CNN
-	1    5700 5150
-	1    0    0    -1
-$EndComp
-Wire Wire Line
-	5500 5200 5300 5200
+P 6450 5150
+F 0 "P3" H 6450 5300 50  0000 C CNN
+F 1 "CONN_01X02" V 6550 5150 50  0000 C CNN
+F 2 "Pin_Headers:Pin_Header_Angled_1x02" H 6450 5150 50  0001 C CNN
+F 3 "" H 6450 5150 50  0000 C CNN
+	1    6450 5150
+	1    0    0    -1
+$EndComp
 Wire Wire Line
 	4150 4400 4950 4400
@@
 L GND #PWR014
 U 1 1 58915A68
-P 5300 5350
-F 0 "#PWR014" H 5300 5100 50  0001 C CNN
-F 1 "GND" H 5300 5200 50  0000 C CNN
-F 2 "" H 5300 5350 50  0000 C CNN
-F 3 "" H 5300 5350 50  0000 C CNN
-	1    5300 5350
+P 5400 5550
+F 0 "#PWR014" H 5400 5300 50  0001 C CNN
+F 1 "GND" H 5400 5400 50  0000 C CNN
+F 2 "" H 5400 5550 50  0000 C CNN
+F 3 "" H 5400 5550 50  0000 C CNN
+	1    5400 5550
 	1    0    0    -1
 $EndComp
@@
 	2450 4400 2350 4400
 Connection ~ 2350 4400
+$Comp
+L R R1
+U 1 1 58DDD5BC
+P 6000 5100
+F 0 "R1" V 6080 5100 50  0000 C CNN
+F 1 "10R4" V 6000 5100 50  0000 C CNN
+F 2 "Resistors_SMD:R_0805" V 5930 5100 50  0001 C CNN
+F 3 "" H 6000 5100 50  0000 C CNN
+	1    6000 5100
+	0    1    1    0
+$EndComp
+$Comp
+L C C1
+U 1 1 58DDD671
+P 5750 5250
+F 0 "C1" H 5775 5350 50  0000 L CNN
+F 1 ".1uF" H 5775 5150 50  0000 L CNN
+F 2 "Capacitors_SMD:C_0805" H 5788 5100 50  0001 C CNN
+F 3 "" H 5750 5250 50  0000 C CNN
+	1    5750 5250
+	1    0    0    -1
+$EndComp
+Wire Wire Line
+	5400 5400 5400 5550
+Wire Wire Line
+	6250 5400 6250 5200
+Connection ~ 5750 5400
+Wire Wire Line
+	6250 5100 6150 5100
+Connection ~ 5750 5100
 $EndSCHEMATC
